File: PBA/Central Heating Control PBA/Central Heating Control PBA.kicad_pcb (KiCad board)
At the start: 2 copper layers, 173.4 x 85.5 mm, 158 parts, among them J1 Screw_Terminal_01x03, J10 Screw_Terminal_01x02, J11 Screw_Terminal_01x02, J12 Screw_Terminal_01x02, J13 Screw_Terminal_01x02, J2 Conn_01x11, J3 Screw_Terminal_01x02, J3_DC5V1 Screw_Terminal_01x02, J4 Screw_Terminal_01x02, J4_AC_OUTPUT1 Screw_Terminal_01x02, J5 Screw_Terminal_01x02, J5_AC_INPUT1 Screw_Terminal_01x02, J6 Screw_Terminal_01x02, J7 Screw_Terminal_01x02, J8 Screw_Terminal_01x02, J9 Screw_Terminal_01x02, Q1 BT136-600, Q10 BT136-600, Q11 BC857, Q12 BC857, Q13 BC857, Q14 BC857, Q15 BC857, Q16 BC857, Q17 BC857, Q18 BC857, Q19 BC857, Q2 BT136-600, Q20 BC857, Q21 BC857, Q22 BT136-600, Q3 BT136-600, Q4 BT136-600, Q5 BT136-600, Q6 BT136-600, Q7 BT136-600, Q8 BT136-600, Q9 BT136-600, U1 ESP32_DevKit_V1_DOIT, U10 MOC3083M, U11 MOC3083M, U12 MOC3083M, U13 DS18B20, U14 DHT11, U2 MOC3083M, U3 MOC3083M, U4 MOC3083M, U5 MOC3083M, U6 MOC3083M, U7 MOC3083M, U8 MOC3083M, U9 MOC3083M

Commit message: pba and code update
Signed-off-by: rgw <rgw@marm.pl>
Parts:
- added D12: 1N5819, Diode_SMD:D_SOD-123, F.Cu at (86.0, 96.5)
- added JP12: floor choose, Jumper:SolderJumper-2_P1.3mm_Open_TrianglePad1.0x1.5mm, F.Cu at (101.1, 112.7)
- added REF**: MountingHole_4,5_Pad_Via, MountingHole:MountingHole_4,5_Pad_Via, F.Cu at (140.7, 49.9)
- added REF**: MountingHole_4,5_Pad_Via, MountingHole:MountingHole_4,5_Pad_Via, F.Cu at (110.3, 110.2)
- added REF**: MountingHole_4,5_Pad_Via, MountingHole:MountingHole_4,5_Pad_Via, F.Cu at (50.5, 49.9)
- added REF**: MountingHole_4,5_Pad_Via, MountingHole:MountingHole_4,5_Pad_Via, F.Cu at (182.1, 115.3)
- added REF**: MountingHole_4,5_Pad_Via, MountingHole:MountingHole_4,5_Pad_Via, F.Cu at (203.0, 43.2)
- added REF**: MountingHole_4,5_Pad_Via, MountingHole:MountingHole_4,5_Pad_Via, F.Cu at (50.5, 99.4)
- C12: footprint Capacitor_SMD:C_0201_0603Metric_Pad0.64x0.40mm_HandSolder -> Capacitor_SMD:C_0805_2012Metric_Pad1.18x1.45mm_HandSolder
- D1, D10, D11, D2, D3, D4, D5, D6, D7, D8, D9: value LED_Small -> LED_S; footprint LED_THT:LED_D3.0mm_Clear -> LED_THT:LED_Rectangular_W3.0mm_H2.0mm
- J1: footprint TerminalBlock_MetzConnect:TerminalBlock_MetzConnect_Type086_RT03403HBLC_1x03_P3.81mm_Horizontal -> TerminalBlock_MetzConnect:TerminalBlock_MetzConnect_Type086_RT03403HBLC_1x03_P3.81mm_Horizontal_hole-1.2
- J4_AC_OUTPUT1, J5_AC_INPUT1: footprint TerminalBlock_MetzConnect:TerminalBlock_MetzConnect_Type171_RT13702HBWC_1x02_P7.50mm_Horizontal -> TerminalBlock_MetzConnect:TerminalBlock_MetzConnect_Type101_RT01602HBWC_1x02_P5.08mm_Horizontal
- Q1, Q10, Q2, Q22, Q3, Q4, Q5, Q6, Q7, Q8, Q9: value BT136-600 -> BTA12-600
- Q11, Q12, Q13, Q14, Q15, Q16, Q17, Q18, Q19, Q20, Q21: value BC857 -> BC817
- R10, R11, R2, R3, R4, R5, R53, R6, R7, R8, R9: value 330R -> 240R
- R42, R43, R44, R45, R46, R47, R48, R49, R50, R51, R52: value 680R -> 330R
- RV1, RV10, RV11, RV12, RV2, RV3, RV4, RV5, RV6, RV7, RV8, RV9: footprint Varistor:RV_Disc_D9mm_W3.3mm_P5mm -> Varistor:RV_Disc_D9mm_W3.3mm_P5mm-hole0.9
- U10, U11, U12, U2, U3, U4, U5, U6, U7, U8, U9: footprint Package_DIP:DIP-6_W7.62mm_Socket_LongPads -> Package_DIP:DIP-6_W7.62mm_LongPads_MOC3803
- U13: footprint Package_TO_SOT_THT:TO-92L_Inline -> Package_TO_SOT_THT:TO-92_Inline_W4.0mm_Horizontal_FlatSideDown
- moved R23 8.81 mm to (45.4, 61.6), turned to -90 degrees
- moved R22 8.27 mm to (107.0, 61.6), turned to -90 degrees
- moved R27 8.27 mm to (121.6, 61.6), turned to -90 degrees
- moved R28 8.26 mm to (136.2, 61.6), turned to -90 degrees
- moved R30 8.25 mm to (167.3, 61.6), turned to -90 degrees
- moved R55 8.24 mm to (196.5, 61.6), turned to -90 degrees
- moved R29 8.23 mm to (151.4, 61.6), turned to -90 degrees
- moved R25 8.23 mm to (77.1, 61.6), turned to -90 degrees
- moved R24 8.22 mm to (62.5, 61.6), turned to -90 degrees
- moved R26 8.22 mm to (91.7, 61.6), turned to -90 degrees
- moved R31 8.22 mm to (182.5, 61.6), turned to -90 degrees
- moved R13 7.90 mm to (45.4, 74.3)
- moved R16 7.40 mm to (91.8, 74.3)
- moved R18 7.29 mm to (136.2, 74.3)
- moved R12 7.28 mm to (107.0, 74.3)
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Connections:
- C10 pad 2: Net-(C1-Pad2) -> Net-(C10-Pad2)
- C11 pad 2: Net-(C1-Pad2) -> Net-(C11-Pad2)
- C12 pad 1: +3V3 -> GNDREF
- C12 pad 2: GNDREF -> +3V3
- C2 pad 2: Net-(C1-Pad2) -> Net-(C2-Pad2)
- C3 pad 2: Net-(C1-Pad2) -> Net-(C3-Pad2)
- C4 pad 2: Net-(C1-Pad2) -> Net-(C4-Pad2)
- C5 pad 2: Net-(C1-Pad2) -> Net-(C5-Pad2)
- C6 pad 2: Net-(C1-Pad2) -> Net-(C6-Pad2)
- C7 pad 2: Net-(C1-Pad2) -> Net-(C7-Pad2)
- C8 pad 2: Net-(C1-Pad2) -> Net-(C8-Pad2)
- C9 pad 2: Net-(C1-Pad2) -> Net-(C9-Pad2)
- D1 pad 1: GNDREF -> Net-(D1-Pad1)
- D10 pad 1: GNDREF -> Net-(D10-Pad1)
- D11 pad 1: GNDREF -> Net-(D11-Pad1)
- D2 pad 1: GNDREF -> Net-(D2-Pad1)
- D3 pad 1: GNDREF -> Net-(D3-Pad1)
- D4 pad 1: GNDREF -> Net-(D4-Pad1)
- D5 pad 1: GNDREF -> Net-(D5-Pad1)
- D6 pad 1: GNDREF -> Net-(D6-Pad1)
- D7 pad 1: GNDREF -> Net-(D7-Pad1)
- D8 pad 1: GNDREF -> Net-(D8-Pad1)
- D9 pad 1: GNDREF -> Net-(D9-Pad1)
- F1 pad 2: Net-(C1-Pad2) -> LINE
- J10 pad 2: Net-(J10-Pad2) -> Net-(C8-Pad2)
- J11 pad 2: Net-(J11-Pad2) -> Net-(C9-Pad2)
- J12 pad 2: Net-(J12-Pad2) -> Net-(C10-Pad2)
- J13 pad 2: Net-(J13-Pad2) -> Net-(C11-Pad2)
- J3 pad 2: Net-(J3-Pad2) -> Net-(C2-Pad2)
- J4 pad 2: Net-(J4-Pad2) -> Net-(C3-Pad2)
- J4_AC_OUTPUT1 pad 2: Net-(C1-Pad2) -> LINE
- J5 pad 2: Net-(J5-Pad2) -> Net-(C4-Pad2)
- J6 pad 2: Net-(J6-Pad2) -> Net-(C5-Pad2)
- J7 pad 2: Net-(J7-Pad2) -> Net-(C1-Pad2)
- J8 pad 2: Net-(J8-Pad2) -> Net-(C6-Pad2)
- J9 pad 2: Net-(J9-Pad2) -> Net-(C7-Pad2)
- JP1 pad 1: Net-(J3-Pad2) -> Net-(C2-Pad2)
- JP1 pad 2: Net-(C1-Pad2) -> LINE
- JP10 pad 1: Net-(J12-Pad2) -> Net-(C10-Pad2)
- JP10 pad 2: Net-(C1-Pad2) -> LINE
- JP11 pad 1: Net-(J13-Pad2) -> Net-(C11-Pad2)
- JP11 pad 2: Net-(C1-Pad2) -> LINE
- JP2 pad 1: Net-(J4-Pad2) -> Net-(C3-Pad2)
- JP2 pad 2: Net-(C1-Pad2) -> LINE
- JP3 pad 1: Net-(J5-Pad2) -> Net-(C4-Pad2)
- JP3 pad 2: Net-(C1-Pad2) -> LINE
- JP4 pad 1: Net-(J7-Pad2) -> Net-(C1-Pad2)
- JP4 pad 2: Net-(C1-Pad2) -> LINE
- JP5 pad 1: Net-(J8-Pad2) -> Net-(C6-Pad2)
- JP5 pad 2: Net-(C1-Pad2) -> LINE
- JP6 pad 1: Net-(J9-Pad2) -> Net-(C7-Pad2)
- JP6 pad 2: Net-(C1-Pad2) -> LINE
- JP7 pad 1: Net-(J10-Pad2) -> Net-(C8-Pad2)
- JP7 pad 2: Net-(C1-Pad2) -> LINE
- JP8 pad 1: Net-(J11-Pad2) -> Net-(C9-Pad2)
- JP8 pad 2: Net-(C1-Pad2) -> LINE
- JP9 pad 1: Net-(J6-Pad2) -> Net-(C5-Pad2)
- JP9 pad 2: Net-(C1-Pad2) -> LINE
- PS1 pad 1: Net-(C1-Pad2) -> LINE
- Q1 pad 1: Net-(J3-Pad2) -> Net-(C2-Pad2)
- Q1 pad 2: Net-(C1-Pad2) -> LINE
- Q10 pad 1: Net-(J12-Pad2) -> Net-(C10-Pad2)
- Q10 pad 2: Net-(C1-Pad2) -> LINE
- Q11 pad 2: +5V -> GNDREF
- Q12 pad 2: +5V -> GNDREF
- Q13 pad 2: +5V -> GNDREF
- Q14 pad 2: +5V -> GNDREF
- Q15 pad 2: +5V -> GNDREF
- Q16 pad 2: +5V -> GNDREF
- Q17 pad 2: +5V -> GNDREF
- Q18 pad 2: +5V -> GNDREF
- Q19 pad 2: +5V -> GNDREF
- Q2 pad 1: Net-(J4-Pad2) -> Net-(C3-Pad2)
- Q2 pad 2: Net-(C1-Pad2) -> LINE
- Q20 pad 2: +5V -> GNDREF
- Q21 pad 2: +5V -> GNDREF
- Q22 pad 1: Net-(J13-Pad2) -> Net-(C11-Pad2)
- Q22 pad 2: Net-(C1-Pad2) -> LINE
- Q3 pad 1: Net-(J5-Pad2) -> Net-(C4-Pad2)
- Q3 pad 2: Net-(C1-Pad2) -> LINE
- Q4 pad 1: Net-(J6-Pad2) -> Net-(C5-Pad2)
- Q4 pad 2: Net-(C1-Pad2) -> LINE
- Q5 pad 1: Net-(J7-Pad2) -> Net-(C1-Pad2)
- Q5 pad 2: Net-(C1-Pad2) -> LINE
- Q6 pad 1: Net-(J8-Pad2) -> Net-(C6-Pad2)
- Q6 pad 2: Net-(C1-Pad2) -> LINE
- Q7 pad 1: Net-(J9-Pad2) -> Net-(C7-Pad2)
- Q7 pad 2: Net-(C1-Pad2) -> LINE
- Q8 pad 1: Net-(J10-Pad2) -> Net-(C8-Pad2)
- Q8 pad 2: Net-(C1-Pad2) -> LINE
- Q9 pad 1: Net-(J11-Pad2) -> Net-(C9-Pad2)
- Q9 pad 2: Net-(C1-Pad2) -> LINE
- R10 pad 1: Net-(R10-Pad1) -> Net-(D9-Pad2)
- R10 pad 2: Net-(Q17-Pad3) -> +5V
- R11 pad 1: Net-(R11-Pad1) -> Net-(D10-Pad2)
- R11 pad 2: Net-(Q14-Pad3) -> +5V
- R2 pad 1: Net-(Q16-Pad3) -> +5V
- R2 pad 2: Net-(R2-Pad2) -> Net-(D1-Pad2)
- R22 pad 1: Net-(C1-Pad1) -> LINE
- R22 pad 2: Net-(J7-Pad2) -> Net-(C1-Pad1)
- R23 pad 1: Net-(C2-Pad1) -> LINE
- R23 pad 2: Net-(J3-Pad2) -> Net-(C2-Pad1)
- R24 pad 1: Net-(C3-Pad1) -> LINE
- R24 pad 2: Net-(J4-Pad2) -> Net-(C3-Pad1)
- R25 pad 1: Net-(C4-Pad1) -> LINE
- R25 pad 2: Net-(J5-Pad2) -> Net-(C4-Pad1)
- R26 pad 1: Net-(C5-Pad1) -> LINE
- R26 pad 2: Net-(J6-Pad2) -> Net-(C5-Pad1)
- R27 pad 1: Net-(C6-Pad1) -> LINE
- R27 pad 2: Net-(J8-Pad2) -> Net-(C6-Pad1)
- R28 pad 1: Net-(C7-Pad1) -> LINE
- R28 pad 2: Net-(J9-Pad2) -> Net-(C7-Pad1)
- R29 pad 1: Net-(C8-Pad1) -> LINE
- R29 pad 2: Net-(J10-Pad2) -> Net-(C8-Pad1)
- R3 pad 1: Net-(Q11-Pad3) -> +5V
- R3 pad 2: Net-(R3-Pad2) -> Net-(D2-Pad2)
- R30 pad 1: Net-(C9-Pad1) -> LINE
- R30 pad 2: Net-(J11-Pad2) -> Net-(C9-Pad1)
- R31 pad 1: Net-(C10-Pad1) -> LINE
- R31 pad 2: Net-(J12-Pad2) -> Net-(C10-Pad1)
- R32 pad 2: Net-(C1-Pad2) -> Net-(C2-Pad2)
- R33 pad 2: Net-(C1-Pad2) -> Net-(C3-Pad2)
- R34 pad 2: Net-(C1-Pad2) -> Net-(C4-Pad2)
- R35 pad 2: Net-(C1-Pad2) -> Net-(C5-Pad2)
- R37 pad 2: Net-(C1-Pad2) -> Net-(C6-Pad2)
- R38 pad 2: Net-(C1-Pad2) -> Net-(C7-Pad2)
- R39 pad 2: Net-(C1-Pad2) -> Net-(C8-Pad2)
- R4 pad 1: Net-(Q12-Pad3) -> +5V
- R4 pad 2: Net-(R4-Pad2) -> Net-(D3-Pad2)
- R40 pad 2: Net-(C1-Pad2) -> Net-(C9-Pad2)
- R41 pad 2: Net-(C1-Pad2) -> Net-(C10-Pad2)
- R5 pad 1: Net-(Q13-Pad3) -> +5V
- R5 pad 2: Net-(R5-Pad2) -> Net-(D4-Pad2)
- R53 pad 1: Net-(R53-Pad1) -> Net-(D11-Pad2)
- R53 pad 2: Net-(Q15-Pad3) -> +5V
- R55 pad 1: Net-(C11-Pad1) -> LINE
- R55 pad 2: Net-(J13-Pad2) -> Net-(C11-Pad1)
- R56 pad 2: Net-(C1-Pad2) -> Net-(C11-Pad2)
- R57 pad 1: Net-(U1-Pad20) -> Net-(R57-Pad1)
- R6 pad 1: Net-(R6-Pad1) -> Net-(D5-Pad2)
- R6 pad 2: Net-(Q18-Pad3) -> +5V
- R7 pad 1: Net-(R7-Pad1) -> Net-(D6-Pad2)
- R7 pad 2: Net-(Q21-Pad3) -> +5V
- R8 pad 1: Net-(R8-Pad1) -> +5V
- R8 pad 2: Net-(Q19-Pad3) -> Net-(D7-Pad2)
- R9 pad 1: Net-(R9-Pad1) -> +5V
- R9 pad 2: Net-(Q20-Pad3) -> Net-(D8-Pad2)
- RV1 pad 1: Net-(C1-Pad2) -> NEUT
- RV1 pad 2: Net-(J3-Pad2) -> Net-(C2-Pad2)
- RV10 pad 1: Net-(C1-Pad2) -> NEUT
- RV10 pad 2: Net-(J12-Pad2) -> Net-(C10-Pad2)
- RV11 pad 1: Net-(C1-Pad2) -> NEUT
- RV11 pad 2: Net-(J13-Pad2) -> Net-(C11-Pad2)
- RV12 pad 2: Net-(C1-Pad2) -> LINE
- RV2 pad 1: Net-(C1-Pad2) -> NEUT
- RV2 pad 2: Net-(J4-Pad2) -> Net-(C3-Pad2)
- RV3 pad 1: Net-(C1-Pad2) -> NEUT
- RV3 pad 2: Net-(J5-Pad2) -> Net-(C4-Pad2)
- RV4 pad 1: Net-(C1-Pad2) -> NEUT
- RV4 pad 2: Net-(J6-Pad2) -> Net-(C5-Pad2)
- RV5 pad 1: Net-(C1-Pad2) -> NEUT
- RV5 pad 2: Net-(J7-Pad2) -> Net-(C1-Pad2)
- RV6 pad 1: Net-(C1-Pad2) -> NEUT
- RV6 pad 2: Net-(J8-Pad2) -> Net-(C6-Pad2)
- RV7 pad 1: Net-(C1-Pad2) -> NEUT
- RV7 pad 2: Net-(J9-Pad2) -> Net-(C7-Pad2)
- RV8 pad 1: Net-(C1-Pad2) -> NEUT
- RV8 pad 2: Net-(J10-Pad2) -> Net-(C8-Pad2)
- RV9 pad 1: Net-(C1-Pad2) -> NEUT
- RV9 pad 2: Net-(J11-Pad2) -> Net-(C9-Pad2)
- U1 pad 12: Net-(J2-Pad3) -> unconnected-(U1-Pad12)
- U1 pad 15: +5V -> Net-(D12-Pad1)
- U1 pad 20: Net-(U1-Pad20) -> unconnected-(U1-Pad20)
- U1 pad 23: unconnected-(U1-Pad23) -> Net-(R57-Pad1)
- U1 pad 24: unconnected-(U1-Pad24) -> Net-(JP12-Pad2)
- U1 pad 25: unconnected-(U1-Pad25) -> Net-(J2-Pad3)
- U10 pad 1: Net-(R10-Pad1) -> Net-(D9-Pad1)
- U10 pad 2: Net-(D9-Pad2) -> Net-(Q17-Pad3)
- U11 pad 1: Net-(R11-Pad1) -> Net-(D10-Pad1)
- U11 pad 2: Net-(D10-Pad2) -> Net-(Q14-Pad3)
- U12 pad 1: Net-(R53-Pad1) -> Net-(D11-Pad1)
- U12 pad 2: Net-(D11-Pad2) -> Net-(Q15-Pad3)
- U14 pad 2: Net-(U1-Pad20) -> Net-(R57-Pad1)
- U2 pad 1: Net-(R2-Pad2) -> Net-(D1-Pad1)
- U2 pad 2: Net-(D1-Pad2) -> Net-(Q16-Pad3)
- U3 pad 1: Net-(R3-Pad2) -> Net-(D2-Pad1)
- U3 pad 2: Net-(D2-Pad2) -> Net-(Q11-Pad3)
- U4 pad 1: Net-(R4-Pad2) -> Net-(D3-Pad1)
- U4 pad 2: Net-(D3-Pad2) -> Net-(Q12-Pad3)
- U5 pad 1: Net-(R5-Pad2) -> Net-(D4-Pad1)
- U5 pad 2: Net-(D4-Pad2) -> Net-(Q13-Pad3)
- U6 pad 1: Net-(R6-Pad1) -> Net-(D5-Pad1)
- U6 pad 2: Net-(D5-Pad2) -> Net-(Q18-Pad3)
- U7 pad 1: Net-(R7-Pad1) -> Net-(D6-Pad1)
- U7 pad 2: Net-(D6-Pad2) -> Net-(Q21-Pad3)
- U8 pad 1: Net-(R8-Pad1) -> Net-(D7-Pad1)
- U8 pad 2: Net-(D7-Pad2) -> Net-(Q19-Pad3)
- U9 pad 1: Net-(R9-Pad1) -> Net-(D8-Pad1)
- U9 pad 2: Net-(D8-Pad2) -> Net-(Q20-Pad3)
Routing:
- net Net-(C1-Pad2): track 829.4 -> 30.2 mm
- net LINE: track 18.3 -> 564.8 mm
- net NEUT: track 295.5 -> 471.3 mm
- net Net-(C2-Pad2): track 0.00 -> 64.0 mm
- net GNDREF: track 527.8 -> 588.7 mm
- net Net-(R57-Pad1): track 0.00 -> 44.2 mm
- net +5V: track 329.1 -> 287.1 mm, vias 2 -> 3
- net Net-(U1-Pad20): track 38.5 -> 0.00 mm
- net Net-(C8-Pad2): track 0.00 -> 35.1 mm
- net Net-(C5-Pad1): track 14.6 -> 49.5 mm
- net Net-(C3-Pad2): track 0.00 -> 32.1 mm
- net Net-(C6-Pad2): track 0.00 -> 31.5 mm
- net Net-(C10-Pad2): track 0.00 -> 30.7 mm
- net Net-(C5-Pad2): track 0.00 -> 30.2 mm
- net Net-(C11-Pad2): track 0.00 -> 30.2 mm
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Other:
- outline, holes or cut-outs redrawn
- board text added: "1"
- board text added: "10"
- board text added: "11"
- board text added: "18B20"
- board text added: "2"
- board text added: "3"
- board text added: "4"
- board text added: "5"
- board text added: "6"
- board text added: "7"
- board text added: "8"
- board text added: "9"
- board text added: "DHT"
- board text added: "N LINE"
- board text added: "SEL"
- board text added: "Sterowanie PODŁ. MARM.pl Sp. z o.o. (c)2022 v.2.1"
- board text removed: "Sterowanie PODŁ. MARM.pl Sp. z o.o. (c)2022 v.2"
